Commit message: Change the robot_hand config to standard defined in franka desk

File: model/franka_description/robots/frankaEmikaPandaVirtual.urdf (robot description, URDF)
Before this commit: robot panda, 13 links, 12 joints
Links:
- link panda_finger_virtual: geometry 
Joints:
- joint panda_finger_virtual_joint: axis 0 0 1 -> 0 1 0; origin xyz=0 0 0.1034 rpy=-1.57079632679 0 -0.785398163397 -> xyz=0 0 0.1034 rpy=0 0 -0.785398163397
